File: 50x50.kicad_pcb (KiCad board)
At the start: 4 copper layers, 50 x 50 mm, 78 parts, among them J1 Conn_01x02, J2 Conn_01x02, J3 USB_C_Receptacle_USB2.0_14P, J4 Conn_01x03, J5 Conn_01x04, SW1 Reset, SW2 SW_SPST, U1 W25Q128JVPIQ TR, U2 RP2040, U4 Voltage Regulator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

Commit message: feat: removed via's from pads
Routing:
- net GND: track 69.0 -> 86.7 mm
- net +3V3: track 177.4 -> 179.0 mm
